File: Button PCB Base/base.brd (EAGLE design)
At the start: 68.6 x 55.5 mm, 6 parts

Commit message: Drill FIX
Routing:
- net GND: track 54.3 -> 17.1 mm
- net START: track 85.9 -> 83.1 mm
Other:
- outline, holes or cut-outs redrawn

Commit message: Revision 2 Minor Fixes
Routing:
- net START: track 83.1 -> 81.3 mm
Other:
- board size 68.6 x 55.5 mm -> 68.6 x 56.3 mm
Changed lines of the file:
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@@
 <fusionsync huburn="a.cGVyc29uYWw6dWUyYzhhMjlk" projecturn="a.cGVyc29uYWw6dWUyYzhhMjlkIzIwMTkwMTI3MTcyNjUwODc2" f3durn="urn:adsk.wipprod:dm.lineage:oTH3DZR4Sw--0gmoHyjf8g" pcbguid="9cf5262c-cac9-4e53-a5cc-fcc682916803" lastpulledtime="2019-01-27T08:21:30Z" lastsyncedchangeguid="0102e9f8-c775-4f7f-a9af-36f7ceacbfbd"/>
 <plain>
-<wire x1="65.3892" y1="65.6748" x2="0.4984" y2="65.6748" width="0.254" layer="20"/>
-<wire x1="0.4984" y1="65.6748" x2="-1.27" y2="63.4492" width="0.254" layer="20" curve="90"/>
+<wire x1="65.3892" y1="66.4368" x2="0.8032" y2="66.386" width="0.254" layer="20"/>
+<wire x1="0.8032" y1="66.386" x2="-1.27" y2="63.4492" width="0.254" layer="20" curve="90"/>
 <wire x1="-1.27" y1="63.4492" x2="-1.27" y2="11.7856" width="0.254" layer="20"/>
 <wire x1="-1.27" y1="11.7856" x2="0.508" y2="10.16" width="0.254" layer="20" curve="90"/>
@@
 <wire x1="65.3908" y1="19.8232" x2="67.2812" y2="21.7136" width="0.254" layer="20" curve="90"/>
 <wire x1="67.2812" y1="21.7136" x2="67.2812" y2="63.478" width="0.254" layer="20"/>
-<wire x1="67.2812" y1="63.478" x2="65.3892" y2="65.6748" width="0.254" layer="20" curve="90"/>
+<wire x1="67.2812" y1="63.478" x2="65.3892" y2="66.4368" width="0.254" layer="20" curve="90"/>
 <hole x="20.955" y="22.098" drill="2.54"/>
 <hole x="1.016" y="23.114" drill="2.54"/>
 <hole x="44.7548" y="23.114" drill="3.81"/>
 <hole x="22.098" y="27.0764" drill="2.54"/>
-<hole x="64.77" y="29.21" drill="2.54"/>
+<hole x="64.77" y="30.0228" drill="2.54"/>
 <hole x="54.9656" y="31.6484" drill="3.81"/>
 <hole x="51.6636" y="41.7576" drill="2.54"/>
-<hole x="1.27" y="63.5" drill="2.54"/>
-<hole x="64.77" y="63.5" drill="2.54"/>
+<hole x="1.3716" y="64.1604" drill="2.54"/>
+<hole x="64.77" y="64.2112" drill="2.54"/>
 <hole x="27.5209" y="34.1122" drill="2.54"/>
 <text x="19.05" y="63.5" size="0.8128" layer="25">GND</text>
@@
 <wire x1="36.67125" y1="17.4625" x2="36.5986" y2="17.3576" width="0.1524" layer="1"/>
 <wire x1="40.48125" y1="17.4625" x2="40.5986" y2="17.3576" width="0.1524" layer="1"/>
-<wire x1="64.4525" y1="43.9547" x2="46.5836" y2="61.8236" width="0.1524" layer="1"/>
-<wire x1="64.4525" y1="31.59125" x2="64.4525" y2="43.9547" width="0.1524" layer="1"/>
-<wire x1="60.0583" y1="31.59125" x2="64.4525" y2="31.59125" width="0.1524" layer="1"/>
-<wire x1="51.4604" y1="22.99335" x2="60.0583" y2="31.59125" width="0.1524" layer="1"/>
-<wire x1="49.0728" y1="22.99335" x2="51.4604" y2="22.99335" width="0.1524" layer="1"/>
+<wire x1="64.8589" y1="43.5483" x2="46.5836" y2="61.8236" width="0.1524" layer="1"/>
+<wire x1="64.8589" y1="35.75685" x2="64.8589" y2="43.5483" width="0.1524" layer="1"/>
+<wire x1="52.0954" y1="22.99335" x2="64.8589" y2="35.75685" width="0.1524" layer="1"/>
+<wire x1="49.0728" y1="22.99335" x2="52.0954" y2="22.99335" width="0.1524" layer="1"/>
 <wire x1="44.6532" y1="18.57375" x2="49.0728" y2="22.99335" width="0.1524" layer="1"/>
 <wire x1="39.37" y1="18.57375" x2="43.815" y2="18.57375" width="0.1524" layer="1"/>
